File: board_diagram.brd (EAGLE design)
At the start: 68.6 x 53.3 mm, 11 parts, among them P1 5V

Commit message: Added diodes and capacitors.
Parts:
- added C1: 0uF, AUTODESK_CIRCUITS_BREADBOARD:RADIAL-D11.36MM
- added D2, D3: (no value), AUTODESK_CIRCUITS_BREADBOARD:D-7.5
Connections:
- removed net N$1 (its old number): JP1.1, P1.2, U2.12, U2.AREF, U2.VIN
- removed net N$2 (its old number): JP1.2, P1.1, U2.GND, U2.GND.
- new net N$13: C1.+, D2.C, JP1.1, U2.12, U2.AREF, U2.VIN
- new net N$14: D2.A, P1.2
- new net N$15: C1.-, D3.A, JP1.2, U2.GND, U2.GND.
- new net N$16: D3.C, P1.1
